Commit message: nav2_gps_tutorial

File: black_donut_description/urdf/gps.xacro (robot description, xacro)
@@ -1,5 +1,5 @@
 <?xml version="1.0"?>
 <robot xmlns:xacro="http://www.ros.org/wiki/xacro">
-<joint name="gps_joint" type="fixed">
+<!-- <joint name="gps_joint" type="fixed">
   <parent link="base_link"/>
   <child link="gps_link"/>
@@ -13,34 +13,30 @@
     <material name="blue"/>
   </visual>
-</link>
-<!-- <gazebo reference="gps_link">
-  <sensor type="gps" name="gps_sensor">
-    <update_rate>1.0</update_rate>
-    <gps>
-      <horizontal_fov>1.047</horizontal_fov>
-      <vertical_fov>1.047</vertical_fov>
-      <range>
-        <min>0.0</min>
-        <max>100.0</max>
-        <resolution>0.01</resolution>
-      </range>
-    </gps>
-    <plugin name="gazebo_ros_gps" filename="libhector_gazebo_ros_gps.so">
-      <topicName>gps/fix</topicName>
-      <frameName>gps_link</frameName>
-    </plugin>
-  </sensor>
-</gazebo> -->
-<gazebo reference="gps_link">
-<sensor name="my_gps" type="gps">
-  <!-- ensure the sensor is active (required) -->
+</link> -->
+<gazebo reference="camera_frame">
+       <material>Gazebo/Black</material>
+<sensor name="tb3_gps" type="gps">
   <always_on>true</always_on>
-  <update_rate>30</update_rate>
+  <update_rate>1</update_rate>
+  <pose>0 0 0 0 0 0</pose>
+  <gps>
+    <position_sensing>
+      <horizontal>
+        <noise type="gaussian">
+          <mean>0.0</mean>
+          <stddev>0.01</stddev>
+        </noise>
+      </horizontal>
+      <vertical>
+        <noise type="gaussian">
+          <mean>0.0</mean>
+          <stddev>0.01</stddev>
+        </noise>
+      </vertical>
+    </position_sensing>
+  </gps>
   <plugin name="my_gps_plugin" filename="libgazebo_ros_gps_sensor.so">
     <ros>
-      <!-- publish to /gps/data -->
-      <namespace>/gps</namespace>
-      <remapping>~/out:=data</remapping>
-      <remapping>~/vel:=velocity</remapping>
+      <remapping>~/out:=/gps/fix</remapping>
     </ros>
   </plugin>
