Commit message: camera_turns2box

File: description/urdf/depth_camera.xacro (robot description, xacro)
@@ -7,5 +7,5 @@
     </joint>
     <link name="camera_frame">
-        <visual>
+        <!-- <visual>
             <geometry>
                 <cylinder radius="0.05" length="0.06"/>
@@ -20,15 +20,15 @@
         <xacro:inertial_cylinder mass="0.1" length="0.06" radius="0.05">
             <origin xyz="0 0 0" rpy="0 0 0"/>
-        </xacro:inertial_cylinder>
+        </xacro:inertial_cylinder> -->
     </link>
     <joint name="camera_optical_joint" type="fixed">
         <parent link="camera_frame"/>
         <child link="camera_optical_link"/>
-        <origin xyz="0 0 0" rpy="-1.5707 0 -1.5707"/>
+        <origin xyz="0.12 0 0" rpy="-1.5707 0 -1.5707"/>
     </joint>
     <link name="camera_optical_link">
         <visual>
             <geometry>
-                <cylinder radius="0.05" length="0.06"/>
+                <box size="0.4 0.03 0.02"/>
             </geometry>
             <material name="blue"/>
@@ -36,10 +36,7 @@
         <collision>
             <geometry>
-                <cylinder radius="0.05" length="0.06"/>
+                <box size="0.4 0.03 0.02"/>
             </geometry>
         </collision>
-        <xacro:inertial_cylinder mass="0.1" length="0.06" radius="0.05">
-            <origin xyz="0 0 0" rpy="0 0 0"/>
-        </xacro:inertial_cylinder>
     </link>
     <gazebo reference="camera_frame">

File: description/urdf/gps.xacro (robot description, xacro)
@@ -19,5 +19,5 @@
         </collision>
         <xacro:inertial_cylinder mass="0.1" length="0.06" radius="0.05">
-            <origin xyz="0 0 0" rpy="0 0 0"/>
+            <origin xyz="0.2 0 0" rpy="0 0 0"/>
         </xacro:inertial_cylinder>
     </link>

File: description/urdf/robot.urdf.xacro (robot description, xacro)
@@ -10,3 +10,4 @@
     <xacro:include filename="depth_camera.xacro" />
     <xacro:include filename="gps.xacro" />
+    <!-- <xacro:include filename="imu.xacro" /> -->
 </robot>
