Commit message: imu_OK

File: description/urdf/imu.xacro (robot description, xacro)
@@ -2,5 +2,5 @@
 <robot xmlns:xacro="http://www.ros.org/wiki/xacro" >
     <joint name="imu_joint" type="fixed">
-        <parent link="hat_link"/>
+        <parent link="base_link"/>
         <child link="imu_link"/>
         <origin xyz="0 0 0.175" rpy="0 0 0"/>
@@ -9,5 +9,5 @@
         <visual>
             <geometry>
-                <<box size="0.02 0.02 0.01"/>
+                <box size="0.02 0.02 0.01"/>
             </geometry>
             <material name="red"/>
@@ -15,5 +15,5 @@
         <collision>
             <geometry>
-                <<box size="0.02 0.02 0.01"/>
+                <box size="0.02 0.02 0.01"/>
             </geometry>
         </collision>
@@ -39,2 +39,3 @@
     </sensor>
   </gazebo>
+</robot>

File: description/urdf/robot.urdf.xacro (robot description, xacro)
@@ -10,4 +10,4 @@
     <xacro:include filename="depth_camera.xacro" />
     <xacro:include filename="gps.xacro" />
-    <!-- <xacro:include filename="imu.xacro" /> -->
+    <xacro:include filename="imu.xacro" />
 </robot>
